File: hv_switching_psu.sch (KiCad schematic (older format))
At the start: 18 parts, among them P1 CONN_2, P2 CONN_2, P3 CONN_2, SW1 SWITCH_INV, T1 IRF644PBF, U1 MAX1771

Commit message: Updated design to version 1.1
Parts:
- added P4: CONN_1, symbol CONN_1
- R2: value 1.5M -> 2M
- R3: value 15K -> 18K
Connections:
- net GND: now also P4.1
Changed lines of the file:
@@
-EESchema Schematic File Version 2  date Wed 26 Sep 2012 06:18:08 PM PDT
+EESchema Schematic File Version 2  date Tue 19 Feb 2013 07:21:48 PM PST
 LIBS:power
 LIBS:device
@@
 EELAYER 25  0
 EELAYER END
-$Descr A4 11700 8267
+$Descr A4 11693 8268
 encoding utf-8
 Sheet 1 1
 Title ""
-Date "26 sep 2012"
+Date "20 feb 2013"
 Rev ""
 Comp ""
@@
 P 8900 3650
 F 0 "R3" V 8980 3650 50  0000 C CNN
-F 1 "15K" V 8900 3650 50  0000 C CNN
+F 1 "18K" V 8900 3650 50  0000 C CNN
 	1    8900 3650
 	1    0    0    -1
@@
 P 8900 2000
 F 0 "R2" V 8980 2000 50  0000 C CNN
-F 1 "1.5M" V 8900 2000 50  0000 C CNN
+F 1 "2M" V 8900 2000 50  0000 C CNN
 	1    8900 2000
 	1    0    0    -1
@@
 	1    0    0    -1
 $EndComp
+$Comp
+L CONN_1 P4
+U 1 1 51243742
+P 2000 3600
+F 0 "P4" H 2080 3600 40  0000 L CNN
+F 1 "CONN_1" H 2000 3655 30  0001 C CNN
+	1    2000 3600
+	0    -1   -1   0
+$EndComp
+Wire Wire Line
+	2000 3750 2000 3900
+$Comp
+L GND #PWR018
+U 1 1 51243792
+P 2000 3900
+F 0 "#PWR018" H 2000 3900 30  0001 C CNN
+F 1 "GND" H 2000 3830 30  0001 C CNN
+	1    2000 3900
+	1    0    0    -1
+$EndComp

Commit message: Completed new design.
Parts:
- R1: value 0.10 -> 0.03
- R2: value 2M -> 1M
- R3: value 18K -> 10K
Other:
- note removed: "0.1 Ohms gives current limit of 0.5A \nwith an input voltage of 12V"
Changed lines of the file:
@@
-EESchema Schematic File Version 2  date Tue 19 Feb 2013 07:21:48 PM PST
+EESchema Schematic File Version 2  date Mon 22 Apr 2013 05:00:30 PM PDT
 LIBS:power
 LIBS:device
@@
 LIBS:irf644pbf
 LIBS:hv_switching_psu-cache
-EELAYER 25  0
+EELAYER 27 0
 EELAYER END
 $Descr A4 11693 8268
@@
 Sheet 1 1
 Title ""
-Date "20 feb 2013"
+Date "23 apr 2013"
 Rev ""
 Comp ""
@@
 Comment4 ""
 $EndDescr
-Text Notes 6150 4750 0    60   ~ 0
-0.1  Ohms gives current limit of 0.5A \nwith an input voltage of 12V
 Wire Wire Line
 	2250 2800 4350 2800
@@
 F 0 "#PWR01" H 750 1150 30  0001 C CNN
 F 1 "GND" H 750 1080 30  0001 C CNN
+F 2 "" H 750 1150 60  0001 C CNN
+F 3 "" H 750 1150 60  0001 C CNN
 	1    750  1150
 	1    0    0    -1
@@
 F 0 "#FLG02" H 750 1170 30  0001 C CNN
 F 1 "PWR_FLAG" H 750 1130 30  0000 C CNN
+F 2 "" H 750 900 60  0001 C CNN
+F 3 "" H 750 900 60  0001 C CNN
 	1    750  900
 	1    0    0    -1
@@
 F 0 "#FLG03" H 3950 1670 30  0001 C CNN
 F 1 "PWR_FLAG" H 3950 1630 30  0000 C CNN
+F 2 "" H 3950 1400 60  0001 C CNN
+F 3 "" H 3950 1400 60  0001 C CNN
 	1    3950 1400
 	1    0    0    -1
@@
 F 0 "#PWR04" H 10250 2000 30  0001 C CNN
 F 1 "GND" H 10250 1930 30  0001 C CNN
+F 2 "" H 10250 2000 60  0001 C CNN
+F 3 "" H 10250 2000 60  0001 C CNN
 	1    10250 2000
 	1    0    0    -1
@@
 F 0 "#PWR05" H 9800 2600 30  0001 C CNN
 F 1 "GND" H 9800 2530 30  0001 C CNN
+F 2 "" H 9800 2600 60  0001 C CNN
+F 3 "" H 9800 2600 60  0001 C CNN
 	1    9800 2600
 	1    0    0    -1
@@
 F 0 "#PWR06" H 8900 4150 30  0001 C CNN
 F 1 "GND" H 8900 4080 30  0001 C CNN
+F 2 "" H 8900 4150 60  0001 C CNN
+F 3 "" H 8900 4150 60  0001 C CNN
 	1    8900 4150
 	1    0    0    -1
@@
 F 0 "RV1" H 8900 2850 50  0000 C CNN
 F 1 "50K" H 8900 2950 50  0000 C CNN
+F 2 "" H 8900 2950 60  0001 C CNN
+F 3 "" H 8900 2950 60  0001 C CNN
 	1    8900 2950
 	0    1    1    0
@@
 P 8900 3650
 F 0 "R3" V 8980 3650 50  0000 C CNN
-F 1 "18K" V 8900 3650 50  0000 C CNN
+F 1 "10K" V 8900 3650 50  0000 C CNN
+F 2 "" H 8900 3650 60  0001 C CNN
+F 3 "" H 8900 3650 60  0001 C CNN
 	1    8900 3650
 	1    0    0    -1
@@
 P 8900 2000
 F 0 "R2" V 8980 2000 50  0000 C CNN
-F 1 "2M" V 8900 2000 50  0000 C CNN
+F 1 "1M" V 8900 2000 50  0000 C CNN
+F 2 "" H 8900 2000 60  0001 C CNN
+F 3 "" H 8900 2000 60  0001 C CNN
 	1    8900 2000
 	1    0    0    -1
@@
 F 0 "#PWR07" H 7900 2250 30  0001 C CNN
 F 1 "GND" H 7900 2180 30  0001 C CNN
+F 2 "" H 7900 2250 60  0001 C CNN
+F 3 "" H 7900 2250 60  0001 C CNN
 	1    7900 2250
 	1    0    0    -1
@@
 F 0 "#PWR08" H 6800 4600 30  0001 C CNN
 F 1 "GND" H 6800 4530 30  0001 C CNN
+F 2 "" H 6800 4600 60  0001 C CNN
+F 3 "" H 6800 4600 60  0001 C CNN
 	1    6800 4600
 	1    0    0    -1
@@
 P 6800 4200
 F 0 "R1" V 6880 4200 50  0000 C CNN
-F 1 "0.10" V 6800 4200 50  0000 C CNN
+F 1 "0.03" V 6800 4200 50  0000 C CNN
+F 2 "" H 6800 4200 60  0001 C CNN
+F 3 "" H 6800 4200 60  0001 C CNN
 	1    6800 4200
 	1    0    0    -1
@@
 F 0 "T1" H 6500 3350 60  0000 C CNN
 F 1 "IRF644PBF" V 7100 3000 60  0000 C CNN
+F 2 "" H 6850 2800 60  0001 C CNN
+F 3 "" H 6850 2800 60  0001 C CNN
 	1    6850 2800
 	1    0    0    -1
@@
 F 0 "D1" H 7350 1700 40  0000 C CNN
 F 1 "ES2F" H 7350 1500 40  0000 C CNN
+F 2 "" H 7350 1600 60  0001 C CNN
+F 3 "" H 7350 1600 60  0001 C CNN
 	1    7350 1600
 	1    0    0    -1
@@
 F 0 "#PWR09" H 5100 3850 30  0001 C CNN
 F 1 "GND" H 5100 3780 30  0001 C CNN
+F 2 "" H 5100 3850 60  0001 C CNN
+F 3 "" H 5100 3850 60  0001 C CNN
 	1    5100 3850
 	1    0    0    -1
@@
 F 0 "#PWR010" H 4100 3850 30  0001 C CNN
 F 1 "GND" H 4100 3780 30  0001 C CNN
+F 2 "" H 4100 3850 60  0001 C CNN
+F 3 "" H 4100 3850 60  0001 C CNN
 	1    4100 3850
 	1    0    0    -1
@@
 F 0 "#PWR011" H 3700 3850 30  0001 C CNN
 F 1 "GND" H 3700 3780 30  0001 C CNN
+F 2 "" H 3700 3850 60  0001 C CNN
+F 3 "" H 3700 3850 60  0001 C CNN
 	1    3700 3850
 	1    0    0    -1
@@
 F 0 "#PWR012" H 2550 3200 30  0001 C CNN
 F 1 "GND" H 2550 3130 30  0001 C CNN
+F 2 "" H 2550 3200 60  0001 C CNN
+F 3 "" H 2550 3200 60  0001 C CNN
 	1    2550 3200
 	1    0    0    -1
@@
 F 0 "P2" V 1850 2900 40  0000 C CNN
 F 1 "CONN_2" V 1950 2900 40  0000 C CNN
+F 2 "" H 1900 2900 60  0001 C CNN
+F 3 "" H 1900 2900 60  0001 C CNN
 	1    1900 2900
 	-1   0    0    1
@@
 F 0 "#PWR013" H 4750 2400 30  0001 C CNN
 F 1 "GND" H 4750 2330 30  0001 C CNN
+F 2 "" H 4750 2400 60  0001 C CNN
+F 3 "" H 4750 2400 60  0001 C CNN
 	1    4750 2400
 	1    0    0    -1
@@
 F 0 "#PWR014" H 4350 2400 30  0001 C CNN
 F 1 "GND" H 4350 2330 30  0001 C CNN
+F 2 "" H 4350 2400 60  0001 C CNN
+F 3 "" H 4350 2400 60  0001 C CNN
 	1    4350 2400
 	1    0    0    -1
@@
 F 0 "#PWR015" H 3650 2400 30  0001 C CNN
 F 1 "GND" H 3650 2330 30  0001 C CNN
+F 2 "" H 3650 2400 60  0001 C CNN
+F 3 "" H 3650 2400 60  0001 C CNN
 	1    3650 2400
 	1    0    0    -1
@@
 F 0 "SW1" H 2850 1850 50  0000 C CNN
 F 1 "SWITCH_INV" H 2900 1550 50  0000 C CNN
+F 2 "" H 3050 1700 60  0001 C CNN
+F 3 "" H 3050 1700 60  0001 C CNN
 	1    3050 1700
 	1    0    0    -1
@@
 F 0 "L1" V 6050 1600 40  0000 C CNN
 F 1 "100uH" V 6200 1600 40  0000 C CNN
+F 2 "" H 6100 1600 60  0001 C CNN
+F 3 "" H 6100 1600 60  0001 C CNN
 	1    6100 1600
 	0    1    1    0
@@
 F 0 "#PWR016" H 5450 2400 30  0001 C CNN
 F 1 "GND" H 5450 2330 30  0001 C CNN
+F 2 "" H 5450 2400 60  0001 C CNN
+F 3 "" H 5450 2400 60  0001 C CNN
 	1    5450 2400
 	1    0    0    -1
@@
 F 0 "#PWR017" H 2550 2100 30  0001 C CNN
 F 1 "GND" H 2550 2030 30  0001 C CNN
+F 2 "" H 2550 2100 60  0001 C CNN
+F 3 "" H 2550 2100 60  0001 C CNN
 	1    2550 2100
 	1    0    0    -1
@@
 F 0 "P3" V 10700 1700 40  0000 C CNN
 F 1 "CONN_2" V 10800 1700 40  0000 C CNN
+F 2 "" H 10750 1700 60  0001 C CNN
+F 3 "" H 10750 1700 60  0001 C CNN
 	1    10750 1700
 	1    0    0    -1
@@
 F 0 "P1" V 1850 1800 40  0000 C CNN
 F 1 "CONN_2" V 1950 1800 40  0000 C CNN
+F 2 "" H 1900 1800 60  0001 C CNN
+F 3 "" H 1900 1800 60  0001 C CNN
 	1    1900 1800
 	-1   0    0    -1
@@
 F 0 "C3" H 4800 2100 50  0000 L CNN
 F 1 "100nF" H 4800 1900 50  0000 L CNN
+F 2 "" H 4750 2000 60  0001 C CNN
+F 3 "" H 4750 2000 60  0001 C CNN
 	1    4750 2000
 	1    0    0    -1
@@
 F 0 "C1" H 3750 3600 50  0000 L CNN
 F 1 "100nF" H 3750 3400 50  0000 L CNN
+F 2 "" H 3700 3500 60  0001 C CNN
+F 3 "" H 3700 3500 60  0001 C CNN
 	1    3700 3500
 	1    0    0    -1
@@
 F 0 "C6" H 9850 2300 50  0000 L CNN
 F 1 "100nF, 250V" H 9850 2100 50  0000 L CNN
+F 2 "" H 9800 2200 60  0001 C CNN
+F 3 "" H 9800 2200 60  0001 C CNN
 	1    9800 2200
 	1    0    0    -1
@@
 F 0 "C2" H 4400 2100 50  0000 L CNN
 F 1 "10uF" H 4400 1900 50  0000 L CNN
+F 2 "" H 4350 2000 60  0001 C CNN
+F 3 "" H 4350 2000 60  0001 C CNN
 	1    4350 2000
 	1    0    0    -1
@@
 F 0 "C5" H 7950 2050 50  0000 L CNN
 F 1 "4.7uF, 250V" H 7950 1850 50  0000 L CNN
+F 2 "" H 7900 1950 60  0001 C CNN
+F 3 "" H 7900 1950 60  0001 C CNN
 	1    7900 1950
 	1    0    0    -1
@@
 F 0 "C4" H 5500 2100 50  0000 L CNN
 F 1 "100uF, 20V" H 5500 1900 50  0000 L CNN
+F 2 "" H 5450 2000 60  0001 C CNN
+F 3 "" H 5450 2000 60  0001 C CNN
 	1    5450 2000
 	1    0    0    -1
@@
 F 0 "U1" H 4700 3450 60  0000 C CNN
 F 1 "MAX1771" H 5450 3450 60  0000 C CNN
+F 2 "" H 5100 3000 60  0001 C CNN
+F 3 "" H 5100 3000 60  0001 C CNN
 	1    5100 3000
 	1    0    0    -1
@@
 F 0 "P4" H 2080 3600 40  0000 L CNN
 F 1 "CONN_1" H 2000 3655 30  0001 C CNN
+F 2 "" H 2000 3600 60  0001 C CNN
+F 3 "" H 2000 3600 60  0001 C CNN
 	1    2000 3600
 	0    -1   -1   0
@@
 F 0 "#PWR018" H 2000 3900 30  0001 C CNN
 F 1 "GND" H 2000 3830 30  0001 C CNN
+F 2 "" H 2000 3900 60  0001 C CNN
+F 3 "" H 2000 3900 60  0001 C CNN
 	1    2000 3900
 	1    0    0    -1

Commit message: Modified resistor settings.
Parts:
- R1: value 0.03 -> 0.01
- R3: value 10K -> 15K
Other:
- note removed: "Based on design by Nick de Smith\nhttp://www.desmith.net/NMdS/Electronics/NixiePSU.html"
Changed lines of the file:
@@
-EESchema Schematic File Version 2  date Mon 22 Apr 2013 05:00:30 PM PDT
+EESchema Schematic File Version 2  date Fri 24 May 2013 06:30:06 PM PDT
 LIBS:power
 LIBS:device
@@
 Sheet 1 1
 Title ""
-Date "23 apr 2013"
+Date "25 may 2013"
 Rev ""
 Comp ""
@@
 	1    0    0    -1
 $EndComp
-Text Notes 3550 6550 2    60   ~ 0
-Based on design by Nick de Smith\nhttp://www.desmith.net/NMdS/Electronics/NixiePSU.html
 Text Notes 10850 1450 2    60   ~ 0
 35-150V
@@
 P 8900 3650
 F 0 "R3" V 8980 3650 50  0000 C CNN
-F 1 "10K" V 8900 3650 50  0000 C CNN
+F 1 "15K" V 8900 3650 50  0000 C CNN
 F 2 "" H 8900 3650 60  0001 C CNN
 F 3 "" H 8900 3650 60  0001 C CNN
@@
 P 6800 4200
 F 0 "R1" V 6880 4200 50  0000 C CNN
-F 1 "0.03" V 6800 4200 50  0000 C CNN
+F 1 "0.01" V 6800 4200 50  0000 C CNN
 F 2 "" H 6800 4200 60  0001 C CNN
 F 3 "" H 6800 4200 60  0001 C CNN
