File: with_display/hv_switching_psu.kicad_pcb (KiCad board)
At the start: 2 copper layers, 73.7 x 85 mm, 24 parts, among them K1 CONN_3, P1 CONN_2, P2 CONN_2, P3 CONN_2, P4 CONN_1, SW1 SWITCH_INV, T1 IRF644PBF, U1 MAX1771

Commit message: Re-worked layout for psu with display.
Parts:
- moved MOUNT_HOLE_1 68.6 mm to (157.5, 162.6)
- moved P4 68.6 mm to (88.9, 162.6)
Routing:
- net GND: track 24.8 -> 229.9 mm
- net /PWR_SW: track 119.0 -> 165.6 mm
- net /HV: track 92.3 -> 106.9 mm
- net /PWR: track 22.3 -> 28.6 mm
- net N-0000011: track 37.6 -> 40.1 mm
- net /SHDN: track 44.0 -> 46.4 mm
- net N-0000010: track 47.2 -> 49.2 mm
- net N-000003: track 12.9 -> 14.0 mm
- net N-0000012: track 23.2 -> 24.2 mm
Other:
- net class SHDN added: clearance 0.254, trace_width 0.2032, via_dia 0.889, via_drill 0.635
- board text added: "IO Rodeo Inc. Electrophoresis Power Supply w/ Display v 1.1"
- board text removed: "IO Rodeo Inc. Electrophoresis Power Supply w/ Display v 1.0"
